File: pbx.sch (KiCad schematic (older format))
At the start: 17 parts

Commit message: wired up stuff
Parts:
- added P?: CONN_01X04, symbol CONN_01X04
- added P?: CONN_01X06, symbol CONN_01X06
Connections:
- net at U?.1 (PCLK): now also P?.6 (P6)
- net at U?.10 (Y12): now also P?.2 (T)
- net at U?.11 (Y11): now also P?.3 (R)
- net at U?.12 (Y10): now also P?.2 (T)
- net at U?.13 (Y9): now also P?.3 (R)
- net at U?.14 (Y8): now also P?.2 (T)
- net at U?.15 (X0): now also P?.2 (T)
- net at U?.16 (X1): now also P?.3 (R)
- net at U?.17 (X2): now also P?.2 (T)
- net at U?.18 (X3): now also P?.3 (R)
- net at U?.19 (X4): now also P?.2 (T)
- net at U?.2 (SCLK): now also P?.5 (P5)
- net at U?.20 (X5): now also P?.3 (R)
- net at U?.21 (X6): now also P?.2 (T)
- net at U?.22 (X7): now also P?.3 (R)
- net at U?.23 (X8): now also P?.2 (T)
- net at U?.24 (X9): now also P?.3 (R)
- net at U?.25 (X10): now also P?.2 (T)
- net at U?.26 (X11): now also P?.3 (R)
- net at U?.27 (X12): now also P?.2 (T)
- net at U?.28 (X13): now also P?.3 (R)
- net at U?.29 (X14): now also P?.2 (T)
- net at U?.3 (SIN): now also P?.4 (P4)
- net at U?.30 (X15): now also P?.3 (R)
- net at U?.31 (Y0): now also P?.2 (T)
- net at U?.32 (Y1): now also P?.3 (R)
- net at U?.33 (Y2): now also P?.2 (T)
- net at U?.34 (Y3): now also P?.3 (R)
- net at U?.35 (Y4): now also P?.2 (T)
- net at U?.36 (Y5): now also P?.3 (R)
- net at U?.37 (Y6): now also P?.2 (T)
- net at U?.38 (Y7): now also P?.3 (R)
- net at U?.4 (VSS): now also P?.1 (P1)
- net at U?.41 (VDD): now also P?.2 (P2)
- net at U?.42 (VCC): now also P?.4 (P4)
- net at U?.43 (DGND): now also P?.1 (P1)
- net at U?.44 (SOUT): now also P?.3 (P3)
- net at U?.7 (Y15): now also P?.3 (R)
- net at U?.8 (Y14): now also P?.2 (T)
- net at U?.9 (Y13): now also P?.3 (R)
- net GND: now reaches P?.1 (S)
- net GND: now also P?.1 (S), P?.1 (S), P?.1 (S), P?.1 (S), P?.1 (S), P?.1 (S), P?.1 (S), P?.1 (S), P?.1 (S), P?.1 (S), P?.1 (S), P?.1 (S), P?.1 (S), P?.1 (S), P?.1 (S), P?.2 (P2)
- no-connect marks 0 -> 1
Other:
- moved on the sheet: P?

Commit message: decoupling caps
Parts:
- added C1, C2, C3: 0.1uF, symbol C
Connections:
- net at P?.2 (P2), U?.41 (VDD): now also C2.2
- new net: C1.2, C2.1, C3.1
